Commit message: feat: add sr gripper collision model

File: assets/sr_gripper/sr_gripper.urdf (robot description, URDF)
Before this commit: robot sr_gripper_custom, 5 links, 4 joints
Links:
- added link world
- link base_link: geometry collision dsf_vert contact=false filename=assets/sr_gripper/meshes/collision/link0_dsf1.obj; collision dsf_vert contact=false filename=assets/sr_gripper/meshes/collision/link0_dsf2.obj
- link left_finger_link_1: geometry collision dsf_vert contact=false filename=assets/sr_gripper/meshes/collision/link1_dsf1.obj; visual mesh filename=meshes/visual/link1.obj
- link left_finger_link_2: geometry collision dsf_vert contact=true filename=assets/sr_gripper/meshes/collision/link2_dsf1.obj; visual mesh filename=meshes/visual/link2.obj
- link right_finger_link_1: geometry collision dsf_vert contact=false filename=assets/sr_gripper/meshes/collision/link1_dsf1.obj; visual mesh filename=meshes/visual/link1.obj
- link right_finger_link_2: geometry collision dsf_vert contact=true filename=assets/sr_gripper/meshes/collision/link2_dsf1.obj; collision dsf_vert contact=true filename=assets/sr_gripper/meshes/collision/link2_dsf1.obj
Joints:
- added joint base_joint: type floating, parent world, child base_link, origin xyz=0 0 0 rpy=0 0 0
- joint left_finger_joint_2: axis 0 1 0 -> 0 -1 0
- joint right_finger_joint_2: axis 0 1 0 -> 0 -1 0

File: assets/ur5e/ur5e.urdf (robot description, URDF)
Before this commit: robot ur5e, 19 links, 18 joints
Links:
- link sr_gripper_base_link: geometry collision dsf_vert contact=false filename=assets/sr_gripper/meshes/collision/link0_dsf1.obj; collision dsf_vert contact=false filename=assets/sr_gripper/meshes/collision/link0_dsf2.obj
- link sr_gripper_left_finger_link_1: geometry collision dsf_vert contact=false filename=assets/sr_gripper/meshes/collision/link1_dsf1.obj; visual mesh filename=../sr_gripper/meshes/visual/link1.obj
- link sr_gripper_left_finger_link_2: geometry collision dsf_vert contact=true filename=assets/sr_gripper/meshes/collision/link2_dsf1.obj; visual mesh filename=../sr_gripper/meshes/visual/link2.obj
- link sr_gripper_right_finger_link_1: geometry collision dsf_vert contact=false filename=assets/sr_gripper/meshes/collision/link1_dsf1.obj; visual mesh filename=../sr_gripper/meshes/visual/link1.obj
- link sr_gripper_right_finger_link_2: geometry collision dsf_vert contact=true filename=assets/sr_gripper/meshes/collision/link2_dsf1.obj; visual mesh filename=../sr_gripper/meshes/visual/link2.obj
- link sr_gripper_right_finger_lower_pad: geometry collision dsf_vert contact=true filename=assets/sr_gripper/meshes/collision/link2_dsf1.obj; visual mesh filename=../sr_gripper/meshes/visual/link2.obj
Joints:
- joint sr_gripper_left_finger_joint_2: axis 0 1 0 -> 0 -1 0
- joint sr_gripper_right_finger_joint_2: axis 0 1 0 -> 0 -1 0
